File: board-smt/VNA2.sch (KiCad schematic (older format))
At the start: 61 parts, among them U2 LM339, U3 SA612, U4 SA612, U5 SA612, U6 LM358, U7 LM358

Commit message: Changed pullup resistors to 10k for less supply noise
Parts:
- R36, R37: value 1k -> 10k
Changed lines of the file:
@@
 P 7750 3250
 F 0 "R36" V 7830 3250 50  0000 C CNN
-F 1 "1k" V 7750 3250 50  0000 C CNN
+F 1 "10k" V 7750 3250 50  0000 C CNN
 F 2 "Resistors_SMD:R_0805_HandSoldering" V 7680 3250 50  0001 C CNN
 F 3 "" H 7750 3250 50  0001 C CNN
@@
 P 7800 4300
 F 0 "R37" V 7880 4300 50  0000 C CNN
-F 1 "1k" V 7800 4300 50  0000 C CNN
+F 1 "10k" V 7800 4300 50  0000 C CNN
 F 2 "Resistors_SMD:R_0805_HandSoldering" V 7730 4300 50  0001 C CNN
 F 3 "" H 7800 4300 50  0001 C CNN

Commit message: Added SD card slot, reorganized pins
Parts:
- C10, C11, C12, C13, C17, C18, C19, C20, C21, C22, C23, C24, C32, C33, C8, C9: LCSC (none) -> C49678
- C14, C15, C16: LCSC (none) -> C51207
- C26, C27, C28: LCSC (none) -> C1710
- C29, C30, C31: LCSC (none) -> C1834
- C34, C35, C36: LCSC (none) -> C46653
- L3, L4, L5: LCSC (none) -> C1017
- R10, R36, R37, R7: LCSC (none) -> C17414
- R19, R20, R21, R25, R26, R27, R30, R31, R33: LCSC (none) -> C4310
- R22, R23, R24: LCSC (none) -> C17407
- R28, R29, R32, R41: LCSC (none) -> C17513
- R34, R35: LCSC (none) -> C17514
- U6, U7: LCSC (none) -> C7950
